File: fan_charger.kicad_pcb (KiCad board)
At the start: 2 copper layers, 110 x 26 mm, 84 parts, among them J1 PWR_JACK, J2 USB_C_Receptacle_6P, J3 NTC, J4 BAT, J5 BAT, J6 FAN, J7 LED, J8 UPDI, P1 VBUS, P2 CC1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

Commit message: Update to rev 2
Parts:
- added C25: 100nF, Capacitor_SMD:C_0603_1608Metric, F.Cu at (136.0, 54.1)
- added Q5: DOZ40P02, fan_charger:VSON-8_3.3x3.3mm_P0.65mm_NexFET, F.Cu at (131.9, 54.9)
- added R29: 1K2, Resistor_SMD:R_0603_1608Metric, F.Cu at (130.4, 64.1)
- C1, C2, C3: value 10uF -> 1uF
- Q4: value AO3401 -> DOZ40P02; footprint Package_TO_SOT_SMD:SOT-23 -> fan_charger:VSON-8_3.3x3.3mm_P0.65mm_NexFET
- R22, R23, R28: value 5K1 -> 330R
- R27: renamed from R4; value 15K -> 10K
- R6: value 330R -> 10K
- R7: value 15K -> 20K
- R8: value 150K -> 6K8
- U1: value BQ25185DLH -> BQ25060DQC; footprint fan_charger:WSON-10-1EP_2x2.2mm_P0.5mm_EP0.9x1.5mm -> Package_SON:WSON-10-1EP_2x3mm_P0.5mm_EP0.84x2.4mm
- moved R27 35.4 mm to (141.8, 56.1)
- moved R6 33.0 mm to (106.6, 57.9)
- moved C2 10.2 mm to (141.6, 58.1)
- moved R8 7.20 mm to (132.5, 60.9), turned to -90 degrees
- moved R26 6.24 mm to (150.3, 47.1)
- moved U1 6.01 mm to (137.7, 57.0), turned to -90 degrees
- moved C1 5.90 mm to (140.5, 54.1), turned to 0 degrees
- moved Q4 4.81 mm to (142.1, 48.1), turned to 90 degrees
- moved R7 4.76 mm to (134.8, 57.0), turned to -90 degrees
- moved R5 2.40 mm to (106.6, 59.9)
- moved D2 2.20 mm to (146.0, 49.6), turned to 90 degrees
- moved R4 1.73 mm to (130.4, 60.9), turned to 90 degrees
- moved F1 1.34 mm to (137.0, 50.0)
- moved C3 0.41 mm to (128.9, 55.2)
- moved J1 0.05 mm to (149.5, 49.2)
- renumbered R27 to R4
Connections:
- Q4 pad 1: +12V -> Net-(D2-K)
- Q4 pad 3: /Power Input and Battery/VBUS -> Net-(D2-K)
- R27 pad 1: /MCU/CHG_STAT1 -> GND
- R27 pad 2: VCC -> Net-(U1-ISET)
- R4 pad 1: GND -> Net-(R29-Pad2)
- R4 pad 2: /MCU/~{CHG_CE} -> /Power Input and Battery/TS
- R5 pad 1: /MCU/CHG_STAT2 -> /MCU/CHG_STAT
- R6 pad 2: Net-(U1-ISET) -> /MCU/~{CHG_EN}
- R7 pad 1: GND -> Net-(U1-LDO)
- R7 pad 2: Net-(U1-ILIM/VSET) -> Net-(R7-Pad2)
- R8 pad 1: GND -> Net-(R7-Pad2)
- R8 pad 2: Net-(U1-ILIM/VSET) -> /Power Input and Battery/TS
- U1 pad 1: VCC -> VIN
- U1 pad 10: VIN -> VCC
- U1 pad 2: +BATT -> Net-(U1-ISET)
- U1 pad 3: /MCU/CHG_STAT2 -> GND
- U1 pad 4: /MCU/~{CHG_CE} -> Net-(U1-LDO)
- U1 pad 5: GND -> /Power Input and Battery/TS
- U1 pad 6: /Power Input and Battery/TS -> +BATT
- U1 pad 7: Net-(U1-ILIM/VSET) -> /MCU/~{CHG_EN}
- U1 pad 8: Net-(U1-ISET) -> /MCU/CHG_STAT
- U1 pad 9: /MCU/CHG_STAT1 -> Net-(Q5-G)
- U5 pad 1: /MCU/CHG_STAT2 -> unconnected-(U5-PA2-Pad1)
- U5 pad 18: /MCU/CHG_STAT1 -> /MCU/CHG_STAT
- U5 pad 20: /MCU/~{CHG_CE} -> /MCU/~{CHG_EN}
Routing:
- net /MCU/CHG_STAT1: track 58.9 -> 0.00 mm, vias 2 -> 0
- net /MCU/CHG_STAT: track 0.00 -> 58.1 mm
- net /MCU/~{CHG_EN}: track 0.00 -> 55.5 mm
- net /MCU/~{CHG_CE}: track 55.2 -> 0.00 mm
- net /MCU/CHG_STAT2: track 54.2 -> 0.00 mm
- net /Power Input and Battery/VBUS: track 139.0 -> 114.3 mm
- net Net-(Q5-G): track 0.00 -> 16.9 mm, vias 0 -> 2
- net VCC: track 182.0 -> 195.6 mm, vias 7 -> 8
- net GND: track 67.4 -> 80.2 mm, vias 108 -> 106
- net /Power Input and Battery/TS: track 45.3 -> 53.7 mm
- net Net-(U1-ILIM/VSET): track 8.32 -> 0.00 mm
- net VIN: track 7.73 -> 0.00 mm
- net Net-(U1-LDO): track 0.00 -> 5.01 mm
- net +12V: track 5.70 -> 10.3 mm
- net Net-(R7-Pad2): track 0.00 -> 3.57 mm
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- added copper zone on F.Cu, net /Power Input and Battery/VBUS
- removed copper zone on F.Cu, net +12V
Other:
- board text added: "10K NTC"
- board text added: "Rev 2"
- board text removed: "10K"
- board text removed: "Rev 1"
