File: fan_charger.kicad_sch (KiCad schematic)
At the start: 1 part

Commit message: Update to rev 2
Other:
- sheet MCU ports: added CHG_STAT, ~{CHG_EN}; removed CHG_STAT1, CHG_STAT2, ~{CHG_CE}
- sheet Power Input and Battery ports: added ~{CHG}; removed STAT1, STAT2
