File: mcu.kicad_sch (KiCad schematic)
At the start: 11 parts, among them J8 UPDI, SW1 FAN_ON, SW2 LED_ON, U5 ATtiny1616-M

Commit message: Update to rev 2
Connections:
- net CHG_STAT1 renamed CHG_STAT
- net CHG_STAT2: no longer names the net of U5.1 (PA2)
- net ~{CHG_CE} renamed ~{CHG_EN}
- no-connect marks 1 -> 2
Other:
- moved on the sheet: C19, D3, J8, R22, R23, R24, R25, R28, SW1, SW2, U5
