File: motor_led.kicad_sch (KiCad schematic)
At the start: 37 parts, among them J6 FAN, J7 LED, Q3 2300, U3 DRV8876PWP, U4 TPS61088RHL

Commit message: Update to rev 2
Parts:
- C23, C24: now not fitted; now left out of the parts list
