File: power_battery.kicad_sch (KiCad schematic)
At the start: 34 parts, among them J1 PWR_JACK, J2 USB_C_Receptacle_6P, J3 NTC, J4 BAT, J5 BAT, P1 VBUS, P2 CC1, P3 CC2, P4 GND, Q1 MOT3145G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

Commit message: Update to rev 2
Parts:
- removed Q4: AO3401, Package_TO_SOT_SMD:SOT-23, symbol Device:Q_PMOS_GSD
- removed U1: BQ25185DLH, fan_charger:WSON-10-1EP_2x2.2mm_P0.5mm_EP0.9x1.5mm, symbol fan_charger:BQ25185DLH
- added C25: 100nF, Capacitor_SMD:C_0603_1608Metric, symbol Device:C_Small
- added Q4, Q5: DOZ40P02, fan_charger:VSON-8_3.3x3.3mm_P0.65mm_NexFET, symbol fan_charger:DOZ40P02
- added R29: 1K2, Resistor_SMD:R_0603_1608Metric, symbol Device:R_Small
- added U1: BQ25060DQC, Package_SON:WSON-10-1EP_2x3mm_P0.5mm_EP0.84x2.4mm, symbol fan_charger:BQ25060DQC
- C1, C2, C3: value 10uF -> 1uF
- R27: value 15K -> 10K
- R6: value 330R -> 10K
- R7: value 15K -> 20K
- R8: value 150K -> 6K8
Connections:
- net +12V: now also Q4.4 (G)
- net +BATT: now also Q5.5 (D), U1.6 (BAT)
- net GND: now also C25.2, R29.1, U1.11 (PAD), U1.3 (VSS); no longer R7.1, R8.1
- net TS: now also R4.2, R8.2, U1.5 (TS)
- net VBUS: now also Q4.5 (D)
- net VCC: now also Q5.1 (S), Q5.2 (S), Q5.3 (S), U1.10 (OUT); no longer R4.2
- net VIN: now also U1.1 (IN)
- net ~{CE}: now also R6.2, U1.7 (EN); no longer R27.2
- net at R7.2: now also R8.1; no longer R8.2
- net at D2.1 (K), F1.1: now also Q4.1 (S), Q4.2 (S), Q4.3 (S)
- net STAT1: no longer names the net of R4.1
- net STAT1: now also R29.2
- net STAT2 renamed ~{CHG}
- net ~{CHG}: now also U1.8 (~{CHG})
- new net: R27.2, U1.2 (ISET)
- new net: C25.1, R7.1, U1.4 (LDO)
- new net: Q5.4 (G), U1.9 (BGATE)
Other:
- note added: "Existing DC Jack The existing M7 diode drops 1.1V SS34 diode drops 0.55V Vin is now in below 10.5V (10.35V)"
- note added: "Iset = 1A"
- note added: "NTC 10K B3950 Connector R1 = 26800, R2 = 16200 Set temp window between 10-40 degC"
- note removed: "Connect 10K R if unused"
- note removed: "Existing DC Jack"
- note removed: "Ilim = 1.1A Iset = 0.9A"
- moved on the sheet: C1, C3, C4, D1, F1, F2, F3, J2, J3, J4, J5, P1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
